File: docs/kicad/tank-level-devkit/tank-level-devkit.kicad_sch (KiCad schematic)
At the start: 14 parts, among them J1 JSN-SR04T, Q1 AO3401A, Q2 2N3904, U1 ESP32_DevKit_V1, U2 MT3608

Commit message: Add TP4056 charger symbols and fix KiCad ERC wiring.
Custom tank-level symbols for TP4056, solar panel, and BAT18650 pin layout;
update schematic power types and GND handling; document ERC rules in README.

Co-authored-by: Cursor <cursoragent@cursor.com>
Parts:
- removed BT1: Battery, Package_TO_SOT_SMD:SOT-23-5, symbol Device:Battery
- added BT1: 18650, Connector:Tag-Connect_TC2030-IDC-FP_2x03_P1.27mm_Vertical, symbol tank-level:BAT18650
- added J2: Panel_USB-A_F, symbol tank-level:SOLAR_USB
- added U3: TP4056, symbol tank-level:TP4056
Connections:
- net at C1.1, C2.1, R5.1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: now also U3.5 (OUT+)
- net GND: no longer names the net of C1.2, J1.2 (GND), Q2.1 (E), R4.1, R6.2, U1.2 (GND), U2.2 (IN-), U2.4 (OUT-)
- net GND: now also U3.6 (OUT-)
- new net: J2.1 (+5V), U3.1 (IN+)
- new net: J2.2 (GND), U3.2 (IN-)
- new net: BT1.1 (+), U3.3 (B+)
- new net: BT1.2 (-), U3.4 (B-)

Commit message: Extend KiCad symbols for charger status and ESP pull-up.
Add TP4056 CHRG/STDBY and ESP32 3V3/GPIO33 pins so the schematic can document charging detection without editing wires in the repo.

Co-authored-by: Cursor <cursoragent@cursor.com>
Connections:
- net at J2.1 (+5V): no longer U3.1 (IN+)
- net at J2.2 (GND): now also U3.7 (CHRG); no longer U3.2 (IN-)
Changed lines of the file:
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@@
 		(pin "2"
+		)
+		(pin "8"
+		)
+		(pin "9"
 		)
 		(instances
@@
 		(pin "6"
 		)
-		(instances
+		(pin "7"
+		)
+		(pin "8"
+		)
+		(instances
